File: Neon_5meter_12V/Neon_5meter_12V.kicad_sch (KiCad schematic)
At the start: 48 parts, among them J1 Conn_01x16_Pin, J2 +12V Jack, J3 Conn_01x16_Pin, J4 Blue strip jack, J5 Pink strip Jack, J6 Conn_01x03_Pin, Q1 IRLML2502TRPBF, Q2 IRLML2502TRPBF, Q3 BSS138, Q4 BSS138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

Commit message: updated BOM
Parts:
- C1: footprint (none) -> Capacitor_SMD:C_1206_3216Metric; link (none) -> https://uge-one.com/product/smd-chip-capacitor-size-1206-1u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
- C2: footprint (none) -> Capacitor_THT:CP_Radial_D10.0mm_P5.00mm; link (none) -> https://makerselectronics.com/product/capacitor-470uf-35v-1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
- C3: footprint (none) -> Capacitor_SMD:CP_Elec_10x10.5; link (none) -> https://uge-one.com/product/smd-aluminum-electrolytic-capac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
- D1: footprint (none) -> Diode_SMD:D_SMA; link (none) -> https://uge-one.com/product/smd-schottky-diode-3a-40v-1n582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
- J2: value +12V Jack -> Jack-DC; link (none) -> https://makerselectronics.com/product/dc-power-jack-female-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
- J4: value Blue strip jack -> Jack-DC; link (none) -> https://makerselectronics.com/product/dc-power-jack-female-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
- J5: value Pink strip Jack -> Jack-DC; link (none) -> https://makerselectronics.com/product/dc-power-jack-female-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
- J6: link (none) -> https://microohm-eg.com/product/jst-3-pin-90-degree-male-co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
- L1: footprint (none) -> CD43_Inductor:CD43; link (none) -> https://uge-one.com/product/smd-power-inductor-470uh-4-5x4x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
- Q1, Q2: link (none) -> https://uge-one.com/product/smd-irlml2502trpbf-sot-23-mosfe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
- R16, R17, R18, R3, R6, R7, R8: footprint Resistor_SMD:R_1206_3216Metric_Pad1.30x1.75mm_HandSolder -> Resistor_SMD:R_0805_2012Metric_Pad1.20x1.40mm_HandSolder; link https://makerselectronics.com/product/chip-resistor-smd-10%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 -> https://uge-one.com/product/0805-smd-chip-resistor-10k/?srs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
- R2, R5: link https://uge-one.com/product/smd-chip-resistor-size-1206-220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 -> https://uge-one.com/product/smd-chip-resistor-size-1206-100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
- R4: link https://makerselectronics.com/product/chip-resistor-smd-9-1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 -> https://makerselectronics.com/product/chip-resistor-smd-1k%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
- SW1, SW2: footprint TS-1088-AR02016:SW_TS-1088-AR02016 -> TS_button_3_4_2:TS_button_3_4_2
- U2: link (none) -> https://uge-one.com/product/xl1509-3-3e1-2a-150khz-buck-dc-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
Changed lines of the file:
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@@
 			)
 		)
-		(property "link" "https://uge-one.com/product/smd-chip-resistor-size-1206-220r-ohm/?srsltid=AfmBOoqmkuXwKrfJ3VxJ5AIPn5xc8j2ZOYO0PqRCmSUCAxMBlBADOpRb"
+		(property "link" "https://uge-one.com/product/smd-chip-resistor-size-1206-100r-ohm/"
 			(at 30.48 156.21 90)
 			(effects
@@
 			)
 		)
-		(property "Footprint" ""
+		(property "Footprint" "CD43_Inductor:CD43"
 			(at 78.74 35.56 0)
 			(effects
@@
 			)
 		)
+		(property "link" "https://uge-one.com/product/smd-power-inductor-470uh-4-5x4x3-2mm-cd43/"
+			(at 78.74 35.56 0)
+			(effects
+				(font
+					(size 1.27 1.27)
+				)
+				(hide yes)
+			)
+		)
 		(pin "1"
 		)
@@
 			)
 		)
-		(property "Footprint" "Resistor_SMD:R_1206_3216Metric_Pad1.30x1.75mm_HandSolder"
+		(property "Footprint" "Resistor_SMD:R_0805_2012Metric_Pad1.20x1.40mm_HandSolder"
 			(at 97.282 83.82 90)
 			(effects
@@
 			)
 		)
-		(property "link" "https://makerselectronics.com/product/chip-resistor-smd-10%cf%89-%c2%b15-250mw-1206/"
+		(property "link" "https://uge-one.com/product/0805-smd-chip-resistor-10k/?srsltid=AfmBOorGllG0mYHf8TnX2S13KIvxT3n0IIoJoriv-BR9zB-dGtGjm2Vg"
 			(at 99.06 83.82 0)
 			(effects
@@
 			)
 		)
-		(property "Footprint" ""
+		(property "Footprint" "Diode_SMD:D_SMA"
 			(at 85.09 26.67 0)
 			(effects
@@
 			)
 		)
+		(property "link" "https://uge-one.com/product/smd-schottky-diode-3a-40v-1n5822-ss34-sma/"
+			(at 85.09 26.67 0)
+			(effects
+				(font
+					(size 1.27 1.27)
+				)
+				(hide yes)
+			)
+		)
 		(pin "1"
 		)
@@
 			)
 		)
+		(property "link" "https://microohm-eg.com/product/jst-3-pin-90-degree-male-connector/"
+			(at 195.58 30.48 0)
+			(effects
+				(font
+					(size 1.27 1.27)
+				)
+				(hide yes)
+			)
+		)
 		(pin "2"
 		)
@@
 			)
 		)
-		(property "Footprint" ""
+		(property "Footprint" "Capacitor_SMD:C_1206_3216Metric"
 			(at 43.18 30.48 0)
 			(effects
@@
 			)
 		)
+		(property "link" "https://uge-one.com/product/smd-chip-capacitor-size-1206-1uf/"
+			(at 43.18 30.48 0)
+			(effects
+				(font
+					(size 1.27 1.27)
+				)
+				(hide yes)
+			)
+		)
 		(pin "1"
 		)
@@
 			)
 		)
+		(property "link" "https://uge-one.com/product/smd-irlml2502trpbf-sot-23-mosfet/?srsltid=AfmBOoqixCZKi2_Rw_QPyVd6y4KRdvrHyCsGijRPH4lNedpiwvgNOyGw"
+			(at 46.99 124.46 0)
+			(effects
+				(font
+					(size 1.27 1.27)
+				)
+				(hide yes)
+			)
+		)
 		(pin "3"
 		)
@@
 			)
 		)
-		(property "Footprint" "Resistor_SMD:R_1206_3216Metric_Pad1.30x1.75mm_HandSolder"
+		(property "Footprint" "Resistor_SMD:R_0805_2012Metric_Pad1.20x1.40mm_HandSolder"
 			(at 97.282 121.92 90)
 			(effects
@@
 			)
 		)
-		(property "link" "https://makerselectronics.com/product/chip-resistor-smd-10%cf%89-%c2%b15-250mw-1206/"
+		(property "link" "https://uge-one.com/product/0805-smd-chip-resistor-10k/?srsltid=AfmBOorGllG0mYHf8TnX2S13KIvxT3n0IIoJoriv-BR9zB-dGtGjm2Vg"
 			(at 99.06 121.92 0)
 			(effects
@@
 			)
 		)
-		(property "Value" "Pink strip Jack"
+		(property "Value" "Jack-DC"
 			(at 114.3 24.13 0)
 			(effects
@@
 			)
 		)
+		(property "link" "https://makerselectronics.com/product/dc-power-jack-female-socket-connector-5-5mmx2-1mm/?srsltid=AfmBOooy7mhTTlq198rTgOOBjODubOeCUUqsiDf1LlSihz3m7IWy6fh7"
+			(at 114.3 30.48 0)
+			(effects
+				(font
+					(size 1.27 1.27)
+				)
+				(hide yes)
+			)
+		)
 		(pin "MP"
 		)
@@
 			)
 		)
-		(property "Value" "+12V Jack"
+		(property "Value" "Jack-DC"
 			(at 29.21 74.93 0)
 			(effects
@@
 			)
 		)
+		(property "link" "https://makerselectronics.com/product/dc-power-jack-female-socket-connector-5-5mmx2-1mm/?srsltid=AfmBOooy7mhTTlq198rTgOOBjODubOeCUUqsiDf1LlSihz3m7IWy6fh7"
+			(at 29.21 81.28 0)
+			(effects
+				(font
+					(size 1.27 1.27)
+				)
+				(hide yes)
+			)
+		)
 		(pin "MP"
 		)
@@
 			)
 		)
-		(property "Footprint" "Resistor_SMD:R_1206_3216Metric_Pad1.30x1.75mm_HandSolder"
+		(property "Footprint" "Resistor_SMD:R_0805_2012Metric_Pad1.20x1.40mm_HandSolder"
 			(at 212.598 132.08 90)
 			(effects
@@
 			)
 		)
-		(property "link" "https://makerselectronics.com/product/chip-resistor-smd-10%cf%89-%c2%b15-250mw-1206/"
+		(property "link" "https://uge-one.com/product/0805-smd-chip-resistor-10k/?srsltid=AfmBOorGllG0mYHf8TnX2S13KIvxT3n0IIoJoriv-BR9zB-dGtGjm2Vg"
 			(at 210.82 132.08 0)
 			(effects
@@
 			)
 		)
-		(property "Footprint" "Resistor_SMD:R_1206_3216Metric_Pad1.30x1.75mm_HandSolder"
+		(property "Footprint" "Resistor_SMD:R_0805_2012Metric_Pad1.20x1.40mm_HandSolder"
 			(at 198.628 132.08 90)
 			(effects
@@
 			)
 		)
-		(property "link" "https://makerselectronics.com/product/chip-resistor-smd-10%cf%89-%c2%b15-250mw-1206/"
+		(property "link" "https://uge-one.com/product/0805-smd-chip-resistor-10k/?srsltid=AfmBOorGllG0mYHf8TnX2S13KIvxT3n0IIoJoriv-BR9zB-dGtGjm2Vg"
 			(at 196.85 132.08 0)
 			(effects
@@
 			)
 		)
-		(property "Footprint" ""
+		(property "Footprint" "Capacitor_SMD:CP_Elec_10x10.5"
 			(at 79.7052 55.88 0)
 			(effects
@@
 			)
 		)
+		(property "link" "https://uge-one.com/product/smd-aluminum-electrolytic-capacitor-330uf-50v-1010-5-mm/"
+			(at 78.74 52.07 0)
+			(effects
+				(font
+					(size 1.27 1.27)
+				)
+				(hide yes)
+			)
+		)
 		(pin "1"
 		)
@@
 			)
 		)
+		(property "link" "https://uge-one.com/product/xl1509-3-3e1-2a-150khz-buck-dc-dc-step-down-converter-regulator-ic-smd/?srsltid=AfmBOoo-d0v4w8P7LjpvPGnwJM-lnyFaeHPU-1Q8rCWLEaeI_F_a5hk3"
+			(at 63.5 29.21 0)
+			(effects
+				(font
+					(size 1.27 1.27)
+				)
+				(hide yes)
+			)
+		)
 		(pin "3"
 		)
@@
 			)
 		)
-		(property "Footprint" "TS-1088-AR02016:SW_TS-1088-AR02016"
+		(property "Footprint" "TS_button_3_4_2:TS_button_3_4_2"
 			(at 191.77 142.24 0)
 			(effects
@@
 			)
 		)
-		(property "link" "https://uge-one.com/product/smd-chip-resistor-size-1206-220r-ohm/?srsltid=AfmBOoqmkuXwKrfJ3VxJ5AIPn5xc8j2ZOYO0PqRCmSUCAxMBlBADOpRb"
+		(property "link" "https://uge-one.com/product/smd-chip-resistor-size-1206-100r-ohm/"
 			(at 30.48 124.46 90)
 			(effects
@@
 			)
 		)
-		(property "Footprint" "Resistor_SMD:R_1206_3216Metric_Pad1.30x1.75mm_HandSolder"
+		(property "Footprint" "Resistor_SMD:R_0805_2012Metric_Pad1.20x1.40mm_HandSolder"
 			(at 35.052 129.54 90)
 			(effects
@@
 			)
 		)
-		(property "link" "https://makerselectronics.com/product/chip-resistor-smd-10%cf%89-%c2%b15-250mw-1206/"
+		(property "link" "https://uge-one.com/product/0805-smd-chip-resistor-10k/?srsltid=AfmBOorGllG0mYHf8TnX2S13KIvxT3n0IIoJoriv-BR9zB-dGtGjm2Vg"
 			(at 36.83 129.54 0)
 			(effects
@@
 			)
 		)
-		(property "Footprint" ""
+		(property "Footprint" "Capacitor_THT:CP_Radial_D10.0mm_P5.00mm"
 			(at 27.6352 35.56 0)
 			(effects
@@
 			)
 		)
+		(property "link" "https://makerselectronics.com/product/capacitor-470uf-35v-1016mm/?srsltid=AfmBOor09AGOe6uRfUPUSJ8gQ4mHe95vw-zHcd40OwpcpkuWNsINe4Bm"
+			(at 26.67 31.75 0)
+			(effects
+				(font
+					(size 1.27 1.27)
+				)
+				(hide yes)
+			)
+		)
 		(pin "1"
 		)
@@
 			)
 		)
-		(property "Footprint" "Resistor_SMD:R_1206_3216Metric_Pad1.30x1.75mm_HandSolder"
+		(property "Footprint" "Resistor_SMD:R_0805_2012Metric_Pad1.20x1.40mm_HandSolder"
 			(at 35.052 161.29 90)
 			(effects
@@
 			)
 		)
-		(property "link" "https://makerselectronics.com/product/chip-resistor-smd-10%cf%89-%c2%b15-250mw-1206/"
+		(property "link" "https://uge-one.com/product/0805-smd-chip-resistor-10k/?srsltid=AfmBOorGllG0mYHf8TnX2S13KIvxT3n0IIoJoriv-BR9zB-dGtGjm2Vg"
 			(at 36.83 161.29 0)
 			(effects
@@
 		(dnp no)
 		(fields_autoplaced yes)
-		(property "Reference" "#PWR08"
+		(property "Reference" "#PWR0101"
 			(at 210.82 95.25 0)
 			(effects
@@
 			(project "Neon_5meter_12V"
 				(path "/bf996e64-b02c-4333-a24f-d261c8c5246e"
-					(reference "#PWR08")
+					(reference "#PWR0101")
 					(unit 1)
 				)
@@
 			)
 		)
-		(property "Footprint" "TS-1088-AR02016:SW_TS-1088-AR02016"
+		(property "Footprint" "TS_button_3_4_2:TS_button_3_4_2"
 			(at 205.74 142.24 0)
 			(effects
@@
 			)
 		)
-		(property "Value" "Blue strip jack"
+		(property "Value" "Jack-DC"
 			(at 152.4 24.13 0)
 			(effects
@@
 			)
 		)
+		(property "link" "https://makerselectronics.com/product/dc-power-jack-female-socket-connector-5-5mmx2-1mm/?srsltid=AfmBOooy7mhTTlq198rTgOOBjODubOeCUUqsiDf1LlSihz3m7IWy6fh7"
+			(at 152.4 30.48 0)
+			(effects
+				(font
+					(size 1.27 1.27)
+				)
+				(hide yes)
+			)
+		)
 		(pin "MP"
 		)
@@
 			)
 		)
-		(property "Footprint" "Resistor_SMD:R_1206_3216Metric_Pad1.30x1.75mm_HandSolder"
+		(property "Footprint" "Resistor_SMD:R_0805_2012Metric_Pad1.20x1.40mm_HandSolder"
 			(at 97.282 104.14 90)
 			(effects
@@
 			)
 		)
-		(property "link" "https://makerselectronics.com/product/chip-resistor-smd-10%cf%89-%c2%b15-250mw-1206/"
+		(property "link" "https://uge-one.com/product/0805-smd-chip-resistor-10k/?srsltid=AfmBOorGllG0mYHf8TnX2S13KIvxT3n0IIoJoriv-BR9zB-dGtGjm2Vg"
 			(at 99.06 104.14 0)
 			(effects
@@
 			)
 		)
+		(property "link" "https://uge-one.com/product/smd-irlml2502trpbf-sot-23-mosfet/?srsltid=AfmBOoqixCZKi2_Rw_QPyVd6y4KRdvrHyCsGijRPH4lNedpiwvgNOyGw"
+			(at 46.99 156.21 0)
+			(effects
+				(font
+					(size 1.27 1.27)
+				)
+				(hide yes)
+			)
+		)
 		(pin "3"
 		)
@@
 			)
 		)
-		(property "link" "https://makerselectronics.com/product/chip-resistor-smd-9-1k%cf%89-%c2%b15-250mw-1206/"
+		(property "link" "https://makerselectronics.com/product/chip-resistor-smd-1k%cf%89-%c2%b15-0-25w-%c2%b1100ppm-%e2%84%83-1206-chip/"
 			(at 210.82 72.39 0)
 			(effects
